File: hardware/osilloscopen.kicad_pcb (KiCad board)
At the start: 2 copper layers, 190 x 30 mm, 60 parts, among them J1 SWO, J10 Conn_01x01_Male, J11 Conn_01x02_Male, J12 Conn_01x03_Male, J13 Conn_01x02_Male, J14 Conn_01x02_Male, J15 Conn_01x01_Male, J16 Conn_01x03_Male, J17 OLED, J18 GND, J19 VBAT, J2 OLED, J3 tip, J4 power, J5 Conn_01x03_Male, J6 Conn_01x01_Male, J7 Conn_01x04_Male, J8 Conn_01x01_Male, J9 Conn_01x03_Male, SW1 SW_Push, SW2 SW_Push, SW3 SW_Push, SW4 SW_Push, SW5 POWER, SW6 RESET, U1 AD623AN, U2 ICL7660, U3 STM32F103C8Tx, U4 AP1117-33, U5 XXX, Y1 Crystal

Commit message: Add files via upload
Parts:
- added MH2: MountingHole, MountingHole:MountingHole_3.5mm, F.Cu at (97.2, 83.8)
- added MH3: MountingHole, MountingHole:MountingHole_3.5mm, F.Cu at (269.2, 83.8)
- added MH4: MountingHole, MountingHole:MountingHole_3.5mm, F.Cu at (269.2, 104.1)
- J1: value SWO -> SWD
- U3: moved to B.Cu
- moved REF** 40.6 mm to (216.1, 108.8)
- moved L1 38.9 mm to (172.7, 86.6), turned to 270 degrees
- moved C4 29.9 mm to (176.5, 86.4), turned to 90 degrees
- moved C3 24.2 mm to (181.6, 86.4), turned to 90 degrees
- moved J11 21.6 mm to (196.8, 81.9)
- moved J10 21.6 mm to (194.3, 81.9)
- moved J14 21.6 mm to (201.9, 81.9)
- moved J19 21.0 mm to (191.8, 103.5)
- moved J15 19.1 mm to (207.0, 81.9)
- moved R13 18.6 mm to (177.0, 100.6), turned to 90 degrees
- moved J13 17.9 mm to (196.8, 99.7)
- moved R12 17.6 mm to (151.6, 83.1), turned to 270 degrees
- moved J9 17.3 mm to (191.8, 99.7), turned to 270 degrees
- moved R15 16.2 mm to (155.2, 83.1)
- moved J5 16.1 mm to (186.7, 81.9), turned to 90 degrees
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Connections:
- net Net-(C3-Pad1) renamed /VDDA
- J19 pad 1: Net-(J19-Pad1) -> (no net)
- U1 pad 1: Net-(U1-Pad1) -> (no net)
- U1 pad 8: Net-(U1-Pad8) -> (no net)
- U2 pad 1: Net-(U2-Pad1) -> (no net)
- U2 pad 6: Net-(U2-Pad6) -> (no net)
- U2 pad 7: Net-(U2-Pad7) -> (no net)
- U3 pad 44: Net-(U3-Pad44) -> (no net)
- U5 pad 1: Net-(U5-Pad1) -> (no net)
- U5 pad 5: Net-(U5-Pad5) -> (no net)
- U5 pad 8: Net-(U5-Pad8) -> (no net)
Routing:
- net VDD: track 323.5 -> 356.2 mm, vias 0 -> 3
- net GNDREF: track 627.9 -> 597.1 mm, vias 14 -> 4
- net /SWDIO: track 25.3 -> 7.99 mm
- net /SWCLK: track 26.0 -> 12.2 mm
- net /KEY3: track 42.7 -> 56.0 mm, vias 0 -> 1
- net /KEY4: track 54.0 -> 66.8 mm, vias 0 -> 1
- net /PA9: track 15.8 -> 5.23 mm
- net /KEY1: track 19.9 -> 30.1 mm, vias 0 -> 1
- net /KEY2: track 31.4 -> 40.8 mm, vias 0 -> 1
- net Net-(U1-Pad5): track 37.7 -> 29.7 mm
- net /PA1: track 5.03 -> 12.8 mm
- net /VDDA: track 31.8 -> 24.2 mm, vias 1 -> 0
- net /PB8: track 11.2 -> 3.91 mm
- net /PB15: track 6.38 -> 13.1 mm
- net /PB10: track 12.7 -> 6.49 mm
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Other:
- net class POWER added: clearance 0.2, trace_width 1, via_dia 0.8, via_drill 0.4
